File: hardware/Unknown-Badge/Unknown-Badge.kicad_sch (KiCad schematic)
At the start: 33 parts, among them J1 Conn_02x03_Odd_Even, J2 OLED, SW1 RESET, SW2 SW_SPDT, U1 CH32V003FxPx

Commit message: fest(Hw):PCB_Sch_Update
Parts:
- removed D4, D5: LED_Small, Unknown:LED_S, symbol Device:LED_Small
- removed D8: LED_Small, Unknown:Led_S_S, symbol Device:LED_Small
- removed R8: 220, Resistor_SMD:R_0603_1608Metric, symbol Device:R_Small
- added D4, D5: LED, LED_SMD:LED_0603_1608Metric, symbol Device:LED
- D1: footprint LED_SMD:LED_0201_0603Metric -> LED_SMD:LED_0603_1608Metric; LCSC# C5440628 -> C434424
- D2: footprint LED_SMD:LED_0402_1005Metric -> LED_SMD:LED_0603_1608Metric; LCSC# C434450 -> C434424
Connections:
- net LED4: now also D4.2 (A)
- net LED5: now also D5.2 (A)
- net at R5.1: now also D5.1 (K)
- net at R4.1: now also D4.1 (K)
- net LED8: no longer names the net of U1.3 (PD6)
- no-connect marks 6 -> 7
Other:
- company: (none) -> ElectronicCats
- title: (none) -> UNKNOWN_BADGE
