File: hardware/Unknown-Badge/Unknown-Badge.kicad_pcb (KiCad board)
At the start: 2 copper layers, 45.9 x 70 mm, 33 parts, among them J1 Conn_02x03_Odd_Even, J2 OLED, SW1 RESET, SW2 SW_SPDT, U1 CH32V003FxPx

Commit message: fest(Hw):PCB_Sch_Update
Parts:
- removed D8: LED_Small, Unknown:Led_S_S
- removed R8: 220, Resistor_SMD:R_0603_1608Metric
- added G***: LOGO, Aesthetics:electronic_cats_logo_8x6, B.Cu at (123.6, 44.0)
- added kibuzzard-682F761D: G***, kibuzzard-682F761D, B.Cu at (122.2, 76.6)
- added kibuzzard-682F7670: G***, kibuzzard-682F7670, F.Cu at (93.9, 49.5)
- added kibuzzard-682F777C: G***, kibuzzard-682F777C, B.Cu at (123.5, 48.2)
- C1, C2, R1, R2, R3, R4, R5, R6, R7: moved to B.Cu
- D1: footprint LED_SMD:LED_0201_0603Metric -> LED_SMD:LED_0603_1608Metric
- D2: footprint LED_SMD:LED_0402_1005Metric -> LED_SMD:LED_0603_1608Metric
- D4, D5: value LED_Small -> LED; footprint Unknown:LED_S -> LED_SMD:LED_0603_1608Metric
- moved R2 104.7 mm to (124.0, 52.3)
- moved R4 101.7 mm to (122.2, 62.6)
- moved R6 94.7 mm to (118.7, 54.0)
- moved R3 93.8 mm to (110.2, 47.5), turned to 90 degrees
- moved C1 86.4 mm to (101.5, 49.0), turned to 90 degrees
- moved D2 79.0 mm to (123.4, 52.0)
- moved C2 77.3 mm to (91.2, 49.5), turned to 180 degrees
- moved D4 74.7 mm to (120.8, 62.6)
- moved R7 71.1 mm to (93.3, 53.9), turned to 180 degrees
- moved R1 69.3 mm to (87.7, 52.3), turned to 180 degrees
- moved D3 68.1 mm to (105.9, 49.8), turned to -90 degrees
- moved R5 64.7 mm to (90.5, 62.3)
- moved D1 51.0 mm to (88.2, 52.1)
- moved D5 47.3 mm to (90.8, 62.4)
- moved BT1 22.7 mm to (113.5, 104.9), turned to 90 degrees
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Connections:
- U1 pad 3: /LED8 -> unconnected-(U1-PD6-Pad3)
Routing:
- net +3.3V: track 0.00 -> 76.0 mm, vias 0 -> 1
- net /LEFT: track 0.00 -> 69.1 mm, vias 0 -> 1
- net /RIGHT: track 0.00 -> 65.8 mm, vias 0 -> 1
- net /UP: track 0.00 -> 60.0 mm, vias 0 -> 1
- net /DOWN: track 0.00 -> 55.3 mm, vias 0 -> 1
- net /SCL: track 0.00 -> 45.6 mm, vias 0 -> 1
- net /SDA: track 0.00 -> 42.9 mm, vias 0 -> 1
- net /LED5: track 0.00 -> 40.2 mm, vias 0 -> 1
- net /LED4: track 0.00 -> 28.0 mm, vias 0 -> 1
- net /LED1: track 0.00 -> 27.9 mm, vias 0 -> 1
- net Net-(BT1--): track 0.00 -> 26.3 mm
- net /SWDIO: track 0.00 -> 24.5 mm, vias 0 -> 1
- net /LED2: track 0.00 -> 20.5 mm, vias 0 -> 1
- net /RST: track 0.00 -> 20.0 mm
- net /LED6: track 0.00 -> 16.0 mm, vias 0 -> 2
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- added copper zone on B.Cu, net GND
- added copper zone on F.Cu, net GND
Other:
- board size 45.9 x 70 mm -> 45.9 x 75 mm

Commit message: feat(Hw):3D_Models_Added
Parts:
- moved G*** 8.39 mm to (115.2, 45.0)
- moved kibuzzard-682F777C 7.75 mm to (115.8, 49.1)
Changed lines of the file:
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@@
 		)
 		(embedded_fonts no)
-		(model "${KICAD6_3DMODEL_DIR}/Connector_PinHeader_2.54mm.3dshapes/PinHeader_1x04_P2.54mm_Vertical.wrl"
+		(model "${KIPRJMOD}/Unknown.pretty/3D/128x32-OLED.STEP"
 			(offset
-				(xyz 0 0 0)
+				(xyz 17.75 -3.75 2.5)
 			)
 			(scale
@@
 			)
 			(rotate
-				(xyz 0 0 0)
+				(xyz -0 -0 -0)
 			)
 		)
@@
 				(font
 					(size 0.001 0.001)
+					(thickness 0.15)
 				)
 			)
@@
 				(font
 					(size 0.001 0.001)
+					(thickness 0.15)
 				)
 			)
@@
 			(effects
 				(font
-					(size 1 1)
+					(size 0.6 0.6)
 					(thickness 0.15)
 				)
@@
 			(effects
 				(font
-					(size 1 1)
+					(size 0.6 0.6)
 					(thickness 0.15)
 				)
@@
 			(effects
 				(font
-					(size 1 1)
+					(size 0.6 0.6)
 					(thickness 0.15)
 				)
@@
 			(effects
 				(font
-					(size 1 1)
+					(size 0.6 0.6)
 					(thickness 0.15)
 				)
@@
 			(effects
 				(font
-					(size 1 1)
+					(size 0.6 0.6)
 					(thickness 0.15)
 				)
@@
 			(effects
 				(font
-					(size 1 1)
+					(size 0.6 0.6)
 					(thickness 0.15)
 				)
@@
 			(effects
 				(font
-					(size 1 1)
+					(size 0.6 0.6)
 					(thickness 0.15)
 				)
@@
 	(footprint "Aesthetics:electronic_cats_logo_8x6"
 		(layer "B.Cu")
-		(at 123.59 44 180)
+		(at 115.25 44.95 180)
 		(property "Reference" "G***"
 			(at 0 0 0)
@@
 			(effects
 				(font
-					(size 1.524 1.524)
+					(size 0.6 0.6)
 					(thickness 0.3)
 				)
@@
 			(effects
 				(font
-					(size 1 1)
+					(size 0.6 0.6)
 					(thickness 0.15)
 				)
@@
 			(effects
 				(font
-					(size 1 1)
+					(size 0.6 0.6)
 					(thickness 0.15)
 				)
@@
 			(effects
 				(font
-					(size 1 1)
+					(size 0.6 0.6)
 					(thickness 0.15)
 				)
@@
 			(effects
 				(font
-					(size 1.27 1.27)
+					(size 0.6 0.6)
 					(thickness 0.254)
 				)
@@
 			(effects
 				(font
-					(size 1 1)
+					(size 0.6 0.6)
 					(thickness 0.15)
 				)
@@
 	(footprint "kibuzzard-682F777C"
 		(layer "B.Cu")
-		(at 123.53 48.21 180)
+		(at 115.825 49.075 180)
 		(descr "Generated with KiBuzzard")
 		(tags "kb_params=eyJBbGlnbm1lbnRDaG9pY2UiOiAiQ2VudGVyIiwgIkNhcExlZnRDaG9pY2UiOiAiKCIsICJDYXBSaWdodENob2ljZSI6ICIpIiwgIkZvbnRDb21ib0JveCI6ICJVYnVudHVNb25vLUIiLCAiSGVpZ2h0Q3RybCI6IDAuNSwgIkxheWVyQ29tYm9Cb3giOiAiRi5TaWxrUyIsICJMaW5lU3BhY2luZ0N0cmwiOiAxLjUsICJNdWx0aUxpbmVUZXh0IjogIlYxLjAiLCAiUGFkZGluZ0JvdHRvbUN0cmwiOiAxLjAsICJQYWRkaW5nTGVmdEN0cmwiOiAxLjAsICJQYWRkaW5nUmlnaHRDdHJsIjogMS4wLCAiUGFkZGluZ1RvcEN0cmwiOiAxLjAsICJXaWR0aEN0cmwiOiAwLjcsICJhZHZhbmNlZENoZWNrYm94IjogZmFsc2UsICJpbmxpbmVGb3JtYXRUZXh0Ym94IjogZmFsc2UsICJsaW5lb3ZlclN0eWxlQ2hvaWNlIjogIlNxdWFyZSIsICJsaW5lb3ZlclRoaWNrbmVzc0N0cmwiOiAxfQ==")
@@
 			(effects
 				(font
-					(size 0.001 0.001)
+					(size 0.6 0.6)
+					(thickness 0.15)
 				)
 				(justify mirror)
@@
 				(font
 					(size 0.001 0.001)
+					(thickness 0.15)
 				)
 				(justify mirror)
@@
 			(effects
 				(font
-					(size 1 1)
+					(size 0.6 0.6)
 					(thickness 0.15)
 				)
@@
 			(effects
 				(font
-					(size 1 1)
+					(size 0.6 0.6)
 					(thickness 0.15)
 				)
@@
 			(effects
 				(font
-					(size 0.001 0.001)
+					(size 0.6 0.6)
+					(thickness 0.15)
 				)
 				(justify mirror)
@@
 				(font
 					(size 0.001 0.001)
+					(thickness 0.15)
 				)
 				(justify mirror)
@@
 			(effects
 				(font
-					(size 1 1)
+					(size 0.6 0.6)
 					(thickness 0.15)
 				)
@@
 		(tags "resistor")
 		(property "Reference" "R3"
-			(at 0 1.43 90)
+			(at -2.56 0.045 90)
 			(layer "B.SilkS")
 			(effects
 				(font
-					(size 1 1)
+					(size 0.6 0.6)
 					(thickness 0.15)
 				)

Commit message: feat(Hw):Labels_updated
Parts:
- removed kibuzzard-682F761D: G***, kibuzzard-682F761D
- removed kibuzzard-682F7670: G***, kibuzzard-682F7670
- removed kibuzzard-682F777C: G***, kibuzzard-682F777C
- added kibuzzard-6839DD39: G***, kibuzzard-6839DD39, B.Cu at (94.0, 49.6)
- added kibuzzard-6839DD63: G***, kibuzzard-6839DD63, B.Cu at (115.3, 49.6)
- added kibuzzard-6839DD94: G***, kibuzzard-6839DD94, B.Cu at (122.2, 78.4)
- added kibuzzard-6839DDBA: G***, kibuzzard-6839DDBA, B.Cu at (122.2, 70.7)
- moved J1 2.04 mm to (123.7, 41.6), turned to -90 degrees
- moved G*** 0.44 mm to (115.3, 45.4)
- moved C2 0.23 mm to (91.0, 49.5)
Routing:
- net +3.3V: track 76.0 -> 83.5 mm
- net /SWDIO: track 24.5 -> 21.6 mm
